File: lineFollowerBasic/powerManagement.kicad_sch (KiCad schematic)
At the start: 0 parts

Commit message: Modified MCU Sch: added crystal, capacitors, FTDI conn, power symbols. Modified Power Module: added battery module, new symbol for converter, power symbols.
Parts:
- added BT1: Battery, symbol Device:Battery
- added U2: ~, symbol line_follower_missing_symbols:N7805-1C
Connections:
- new net: BT1.1 (+), U2.1 (+Vin)
- new net +5V: U2.3 (+Vout)
- new net GND: BT1.2 (-), U2.2 (GND)
Changed lines of the file:
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@@
 (kicad_sch (version 20230121) (generator eeschema)
   (paper "A4")
+  (wire (pts (xy 76.835 59.055) (xy 73.025 59.055))
+    (stroke (width 0) (type default))
+  )
+  (wire (pts (xy 73.025 56.515) (xy 76.835 56.515))
+    (stroke (width 0) (type default))
+  )
+  (wire (pts (xy 73.025 74.295) (xy 73.025 73.025))
+    (stroke (width 0) (type default))
+  )
+  (wire (pts (xy 73.025 59.055) (xy 73.025 62.865))
+    (stroke (width 0) (type default))
+  )
+  (wire (pts (xy 73.025 53.975) (xy 76.835 53.975))
+    (stroke (width 0) (type default))
+  )
+  (symbol (lib_id "power:GND") (at 73.025 56.515 270) (unit 1)
+    (in_bom yes) (on_board yes) (dnp no)
+    (property "Reference" "#PWR06" (at 66.675 56.515 0)
+      (effects (font (size 1.27 1.27)) hide)
+    )
+    (property "Value" "GND" (at 69.85 56.515 90)
+      (effects (font (size 1.27 1.27)) (justify right))
+    )
+    (property "Footprint" "" (at 73.025 56.515 0)
+      (effects (font (size 1.27 1.27)) hide)
+    )
+    (property "Datasheet" "" (at 73.025 56.515 0)
+      (effects (font (size 1.27 1.27)) hide)
+    )
+    (pin "1")
+    (instances
+      (project "lineFollowerBasic"
+        (path "/751730cf-cec6-4b73-8a36-3b45eebd4e7c/f40ec953-ba2a-406c-9419-0b14e79f8823"
+          (reference "#PWR06") (unit 1)
+        )
+      )
+    )
+  )
+  (symbol (lib_id "power:GND") (at 73.025 74.295 0) (unit 1)
+    (in_bom yes) (on_board yes) (dnp no) (fields_autoplaced)
+    (property "Reference" "#PWR05" (at 73.025 80.645 0)
+      (effects (font (size 1.27 1.27)) hide)
+    )
+    (property "Value" "GND" (at 73.025 78.74 0)
+      (effects (font (size 1.27 1.27)))
+    )
+    (property "Footprint" "" (at 73.025 74.295 0)
+      (effects (font (size 1.27 1.27)) hide)
+    )
+    (property "Datasheet" "" (at 73.025 74.295 0)
+      (effects (font (size 1.27 1.27)) hide)
+    )
+    (pin "1")
+    (instances
+      (project "lineFollowerBasic"
+        (path "/751730cf-cec6-4b73-8a36-3b45eebd4e7c/f40ec953-ba2a-406c-9419-0b14e79f8823"
+          (reference "#PWR05") (unit 1)
+        )
+      )
+    )
+  )
+  (symbol (lib_id "line_follower_missing_symbols:N7805-1C") (at 83.185 62.865 180) (unit 1)
+    (in_bom yes) (on_board yes) (dnp no)
+    (property "Reference" "U2" (at 87.63 60.325 0)
+      (effects (font (size 1.27 1.27)) (justify right))
+    )
+    (property "Value" "~" (at 83.185 62.865 0)
+      (effects (font (size 1.27 1.27)))
+    )
+    (property "Footprint" "" (at 83.185 62.865 0)
+      (effects (font (size 1.27 1.27)) hide)
+    )
+    (property "Datasheet" "" (at 83.185 62.865 0)
+      (effects (font (size 1.27 1.27)) hide)
+    )
+    (pin "1")
+    (pin "2")
+    (pin "3")
+    (instances
+      (project "lineFollowerBasic"
+        (path "/751730cf-cec6-4b73-8a36-3b45eebd4e7c/f40ec953-ba2a-406c-9419-0b14e79f8823"
+          (reference "U2") (unit 1)
+        )
+      )
+    )
+  )
+  (symbol (lib_id "Device:Battery") (at 73.025 67.945 0) (unit 1)
+    (in_bom yes) (on_board yes) (dnp no) (fields_autoplaced)
+    (property "Reference" "BT1" (at 76.835 66.929 0)
+      (effects (font (size 1.27 1.27)) (justify left))
+    )
+    (property "Value" "Battery" (at 76.835 69.469 0)
+      (effects (font (size 1.27 1.27)) (justify left))
+    )
+    (property "Footprint" "" (at 73.025 66.421 90)
+      (effects (font (size 1.27 1.27)) hide)
+    )
+    (property "Datasheet" "~" (at 73.025 66.421 90)
+      (effects (font (size 1.27 1.27)) hide)
+    )
+    (pin "1")
+    (pin "2")
+    (instances
+      (project "lineFollowerBasic"
+        (path "/751730cf-cec6-4b73-8a36-3b45eebd4e7c/f40ec953-ba2a-406c-9419-0b14e79f8823"
+          (reference "BT1") (unit 1)
+        )
+      )
+    )
+  )
+  (symbol (lib_id "power:+5V") (at 73.025 53.975 90) (unit 1)
+    (in_bom yes) (on_board yes) (dnp no)
+    (property "Reference" "#PWR07" (at 76.835 53.975 0)
+      (effects (font (size 1.27 1.27)) hide)
+    )
+    (property "Value" "+5V" (at 69.85 53.975 90)
+      (effects (font (size 1.27 1.27)) (justify left))
+    )
+    (property "Footprint" "" (at 73.025 53.975 0)
+      (effects (font (size 1.27 1.27)) hide)
+    )
+    (property "Datasheet" "" (at 73.025 53.975 0)
+      (effects (font (size 1.27 1.27)) hide)
+    )
+    (pin "1")
+    (instances
+      (project "lineFollowerBasic"
+        (path "/751730cf-cec6-4b73-8a36-3b45eebd4e7c/f40ec953-ba2a-406c-9419-0b14e79f8823"
+          (reference "#PWR07") (unit 1)
+        )
+      )
+    )
+  )
 )
