File: lineFollowerBasic/sensorArraySubsystem.kicad_sch (KiCad schematic)
At the start: 0 parts

Commit message: Sensors & Multiplexor
Parts:
- added S1, S10, S11, S12, S13, S14, S15, S16, S2, S3, S4, S5, S6, S7, S8, S9: QRE1113, OptoDevice:OnSemi_CASE100AQ, symbol Sensor_Proximity:QRE1113
- added U3: CD74HC4067M, Package_SO:SOIC-24W_7.5x15.4mm_P1.27mm, symbol 74xx:CD74HC4067M
- added U4: ATmega328-P, Package_DIP:DIP-28_W7.62mm, symbol MCU_Microchip_ATmega:ATmega328-P
Connections:
- new net: S4.3, U3.6 (I3)
- new net: S6.3, U3.4 (I5)
- new net: S11.3, U3.21 (I10)
- new net: S10.3, U3.22 (I9)
- new net: U3.13 (S3), U4.11 (PD5)
- new net: U4.22 (GND), U4.8 (GND)
- new net: U3.1 (COM), U4.23 (PC0)
- new net: U3.10 (S0), U4.4 (PD2)
- new net: U3.11 (S1), U4.5 (PD3)
- new net: U3.14 (S2), U4.6 (PD4)
- new net: S3.3, U3.7 (I2)
- new net: S1.3, U3.9 (I0)
- new net: S2.3, U3.8 (I1)
- new net: S8.3, U3.2 (I7)
- new net: S16.3, U3.16 (I15)
- new net: S14.3, U3.18 (I13)
- new net: S7.3, U3.3 (I6)
- new net: S12.3, U3.20 (I11)
- new net: S15.3, U3.17 (I14)
- new net: S13.3, U3.19 (I12)
- new net: S9.3, U3.23 (I8)
- new net: S5.3, U3.5 (I4)

Commit message: Tu mensaje de commit
Connections:
- net +5V: now reaches S4.1 (A)
- net +5V: now also S1.1 (A), S10.1 (A), S11.1 (A), S12.1 (A), S13.1 (A), S14.1 (A), S15.1 (A), S16.1 (A), S2.1 (A), S3.1 (A), S5.1 (A), S6.1 (A), S7.1 (A), S8.1 (A), S9.1 (A), U3.24 (VCC)
- net at S4.3, U3.6 (I3): now also S7.3, U3.3 (I6)
Other:
- moved on the sheet: S1, S10, S11, S12, S13, S14, S15, S16, S2, S3, S4, S5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

Commit message: Deleted extra ATMEGAs, added labels
Parts:
- removed U4: ATmega328-P, Package_DIP:DIP-28_W7.62mm, symbol MCU_Microchip_ATmega:ATmega328-P
Connections:
- net PD5/PWM: now reaches U3.13 (S3)
- net PC0/ADC0: now reaches U3.1 (COM)
- net PD2: now reaches U3.10 (S0)
- net PD3/PWM: now reaches U3.11 (S1)
- net PD4: now reaches U3.14 (S2)
- net GND: now reaches U3.12 (GND)
